Commit message: Cameras implementadas
Signed-off-by: Daniel <da.quinga.2020@alumnos.urjc.es>

File: robot/robot.urdf (robot description, URDF)
Before this commit: robot rover, 16 links, 15 joints
Links:
- added link camera_chasis; visual box size=0.5 0.5 0.5; visual sphere radius=.05
- added link camera_end_effector; visual box size=0.15 0.15 0.15; visual sphere radius=.05
Joints:
- added joint camera_chasis_joint: type fixed, parent base_link, child camera_chasis
- added joint camera_end_effector_joint: type fixed, parent gripper0_link, child camera_end_effector, origin xyz=0 0  0.16 rpy=0 0 0
